Commit message: Switch base, torso, and head to STL meshes; refine kinematics
- Add link_mesh() helper to generator; reference 5 STLs (base_link,
  torso_link, neck_pan_link, neck_tilt_link, camera_link)
- Merge waist_link into torso_link (fixes 30mm Z offset bug at shoulder
  mount and neck)
- Apply CAD-measured dimensions (column 261.5/237.5, shoulder ±71.5,
  arm offsets, gripper kinematics, neck/camera)
- Move shoulder J1->J2 offset to Y direction (was Z), matching the
  outboard-bracket layout of the real robot
- Convert gripper from revolute pivot to parallel prismatic with mimic
- Split PAN->TILT offset into X and Z (was Z-only)
- Refactor camera_link frame to camera body center; sensor-plane offset
  compensated in TILT_TO_CAMERA

Co-Authored-By: Claude Opus 4.7 <noreply@anthropic.com>

File: dual_arm_robot.urdf (robot description, URDF)
Before this commit: robot dual_arm_robot, 32 links, 31 joints
Links:
- removed link waist_link
- link L_finger_left: geometry collision box size=0.01 0.012 0.085; visual box size=0.01 0.012 0.085
- link L_finger_right: geometry collision box size=0.01 0.012 0.085; visual box size=0.01 0.012 0.085
- link L_gripper_base: geometry collision box size=0.04 0.06 0.09; visual box size=0.04 0.06 0.09
- link L_link3: geometry collision cylinder length=0.041 radius=0.022; visual cylinder length=0.041 radius=0.022
- link L_link5: geometry collision cylinder length=0.0405 radius=0.018; visual cylinder length=0.0405 radius=0.018
- link R_finger_left: geometry collision box size=0.01 0.012 0.085; visual box size=0.01 0.012 0.085
- link R_finger_right: geometry collision box size=0.01 0.012 0.085; visual box size=0.01 0.012 0.085
- link R_gripper_base: geometry collision box size=0.04 0.06 0.09; visual box size=0.04 0.06 0.09
- link R_link3: geometry collision cylinder length=0.041 radius=0.022; visual cylinder length=0.041 radius=0.022
- link R_link5: geometry collision cylinder length=0.0405 radius=0.018; visual cylinder length=0.0405 radius=0.018
- link base_link: geometry collision mesh filename=meshes/base_link.stl scale=0.001 0.001 0.001; visual mesh filename=meshes/base_link.stl scale=0.001 0.001 0.001
- link camera_link: geometry collision mesh filename=meshes/camera_link.stl scale=0.001 0.001 0.001; visual mesh filename=meshes/camera_link.stl scale=0.001 0.001 0.001
- link neck_pan_link: mass 0.082 -> 0.1; geometry collision mesh filename=meshes/neck_pan_link.stl scale=0.001 0.001 0.001; visual mesh filename=meshes/neck_pan_link.stl scale=0.001 0.001 0.001
- link neck_tilt_link: mass 0.082 -> 0.1; geometry collision mesh filename=meshes/neck_tilt_link.stl scale=0.001 0.001 0.001; visual mesh filename=meshes/neck_tilt_link.stl scale=0.001 0.001 0.001
- link torso_link: mass 1.5 -> 1.8; geometry collision mesh filename=meshes/torso_link.stl scale=0.001 0.001 0.001; visual mesh filename=meshes/torso_link.stl scale=0.001 0.001 0.001
Joints:
- removed joint torso_fixed
- joint L_gripper_base_fixed: origin xyz=0 0 -0.03 rpy=0 0 0 -> xyz=0 0 0 rpy=0 0 0
- joint L_gripper_joint: limit lower=0 upper=0.05 effort=20 velocity=0.1 -> lower=0 upper=0.037 effort=20 velocity=0.1; origin xyz=0 0.015 -0.04 rpy=0 0 0 -> xyz=0 0.01836 -0.09 rpy=0 0 0
- joint L_gripper_mimic: limit lower=-0.05 upper=0 effort=20 velocity=0.1 -> lower=-0.037 upper=0 effort=20 velocity=0.1; origin xyz=0 -0.015 -0.04 rpy=0 0 0 -> xyz=0 -0.01836 -0.09 rpy=0 0 0
- joint L_joint2: origin xyz=0 0 -0.05 rpy=0 0 0 -> xyz=0 0.06725 0 rpy=0 0 0
- joint L_joint3: origin xyz=0 0 -0.06 rpy=0 0 0 -> xyz=0 0 -0.0805 rpy=0 0 0
- joint L_joint4: origin xyz=0 0 -0.15 rpy=0 0 0 -> xyz=0 0 -0.041 rpy=0 0 0
- joint L_joint5: origin xyz=0 0 -0.04 rpy=0 0 0 -> xyz=0 0 -0.064 rpy=0 0 0
- joint L_joint6: origin xyz=0 0 -0.13 rpy=0 0 0 -> xyz=0 0 -0.0405 rpy=0 0 0
- joint L_joint7: origin xyz=0 0 -0.04 rpy=0 0 0 -> xyz=0 0 -0.028 rpy=0 0 0
- joint L_shoulder_mount_fixed: origin xyz=0 0.11 0.3 rpy=0 0 0 -> xyz=0 0.0715 0.21 rpy=0 0 0
- joint L_tcp_fixed: origin xyz=0 0 -0.1 rpy=0 0 0 -> xyz=0 0 -0.175 rpy=0 0 0
- joint R_gripper_base_fixed: origin xyz=0 0 -0.03 rpy=0 0 0 -> xyz=0 0 0 rpy=0 0 0
- joint R_gripper_joint: limit lower=0 upper=0.05 effort=20 velocity=0.1 -> lower=0 upper=0.037 effort=20 velocity=0.1; origin xyz=0 0.015 -0.04 rpy=0 0 0 -> xyz=0 0.01836 -0.09 rpy=0 0 0
- joint R_gripper_mimic: limit lower=-0.05 upper=0 effort=20 velocity=0.1 -> lower=-0.037 upper=0 effort=20 velocity=0.1; origin xyz=0 -0.015 -0.04 rpy=0 0 0 -> xyz=0 -0.01836 -0.09 rpy=0 0 0
- joint R_joint2: origin xyz=0 0 -0.05 rpy=0 0 0 -> xyz=0 -0.06725 0 rpy=0 0 0
- joint R_joint3: origin xyz=0 0 -0.06 rpy=0 0 0 -> xyz=0 0 -0.0805 rpy=0 0 0
- joint R_joint4: origin xyz=0 0 -0.15 rpy=0 0 0 -> xyz=0 0 -0.041 rpy=0 0 0
- joint R_joint5: origin xyz=0 0 -0.04 rpy=0 0 0 -> xyz=0 0 -0.064 rpy=0 0 0
- joint R_joint6: origin xyz=0 0 -0.13 rpy=0 0 0 -> xyz=0 0 -0.0405 rpy=0 0 0
- joint R_joint7: origin xyz=0 0 -0.04 rpy=0 0 0 -> xyz=0 0 -0.028 rpy=0 0 0
- joint R_shoulder_mount_fixed: origin xyz=0 -0.11 0.3 rpy=0 0 0 -> xyz=0 -0.0715 0.21 rpy=0 0 0
- joint R_tcp_fixed: origin xyz=0 0 -0.1 rpy=0 0 0 -> xyz=0 0 -0.175 rpy=0 0 0
- joint camera_fixed: origin xyz=0 0 0 rpy=0 0 0 -> xyz=0.05195 0 0 rpy=0 0 0
- joint camera_optical_fixed: origin xyz=0.03 0 0 rpy=-1.5708 0 -1.5708 -> xyz=0 0 0 rpy=-1.5708 0 -1.5708
- joint neck_pan_joint: origin xyz=0 0 0.34 rpy=0 0 0 -> xyz=0 0 0.2805 rpy=0 0 0
- joint neck_tilt_joint: origin xyz=0 0 0.04 rpy=0 0 0 -> xyz=0.024 0 0.0195 rpy=0 0 0
- joint waist_joint: child waist_link -> torso_link; origin xyz=0 0 0.18 rpy=0 0 0 -> xyz=0 0 0.2615 rpy=0 0 0

Commit message: Re-measure: J2_TO_J3 82.5mm, drop camera sensor-plane compensation
- J2_TO_J3: 80.5 -> 82.5mm (CAD updated)
- TILT_TO_CAMERA: 51.95 -> 56.25mm: camera STL origin is at the
  sensor plane (not body center), so the prior -4.30mm compensation
  was wrong

Co-Authored-By: Claude Opus 4.7 <noreply@anthropic.com>

File: dual_arm_robot.urdf (robot description, URDF)
Before this commit: robot dual_arm_robot, 31 links, 30 joints
Joints:
- joint L_joint3: origin xyz=0 0 -0.0805 rpy=0 0 0 -> xyz=0 0 -0.0825 rpy=0 0 0
- joint R_joint3: origin xyz=0 0 -0.0805 rpy=0 0 0 -> xyz=0 0 -0.0825 rpy=0 0 0
- joint camera_fixed: origin xyz=0.05195 0 0 rpy=0 0 0 -> xyz=0.05625 0 0 rpy=0 0 0
