Commit message: Add dual-arm STL meshes to URDF

File: dual_arm_robot.urdf (robot description, URDF)
Before this commit: robot dual_arm_robot, 31 links, 30 joints
Links:
- link L_finger_left: geometry collision mesh filename=meshes/L_finger_left.stl scale=0.001 0.001 0.001; visual mesh filename=meshes/L_finger_left.stl scale=0.001 0.001 0.001
- link L_finger_right: geometry collision mesh filename=meshes/L_finger_right.stl scale=0.001 0.001 0.001; visual mesh filename=meshes/L_finger_right.stl scale=0.001 0.001 0.001
- link L_gripper_base: geometry collision mesh filename=meshes/L_gripper_base.stl scale=0.001 0.001 0.001; visual mesh filename=meshes/L_gripper_base.stl scale=0.001 0.001 0.001
- link L_link1: geometry collision mesh filename=meshes/L_link1.stl scale=0.001 0.001 0.001; visual mesh filename=meshes/L_link1.stl scale=0.001 0.001 0.001
- link L_link2: geometry collision mesh filename=meshes/L_link2.stl scale=0.001 0.001 0.001; visual mesh filename=meshes/L_link2.stl scale=0.001 0.001 0.001
- link L_link3: geometry collision mesh filename=meshes/L_link3.stl scale=0.001 0.001 0.001; visual mesh filename=meshes/L_link3.stl scale=0.001 0.001 0.001
- link L_link4: geometry collision mesh filename=meshes/L_link4.stl scale=0.001 0.001 0.001; visual mesh filename=meshes/L_link4.stl scale=0.001 0.001 0.001
- link L_link5: geometry collision mesh filename=meshes/L_link5.stl scale=0.001 0.001 0.001; visual mesh filename=meshes/L_link5.stl scale=0.001 0.001 0.001
- link L_link6: geometry collision mesh filename=meshes/L_link6.stl scale=0.001 0.001 0.001; visual mesh filename=meshes/L_link6.stl scale=0.001 0.001 0.001
- link L_link7: geometry collision mesh filename=meshes/L_link7.stl scale=0.001 0.001 0.001; visual mesh filename=meshes/L_link7.stl scale=0.001 0.001 0.001
- link L_shoulder_mount: mass 0.05 -> None; geometry 
- link R_finger_left: geometry collision mesh filename=meshes/R_finger_left.stl scale=0.001 0.001 0.001; visual mesh filename=meshes/R_finger_left.stl scale=0.001 0.001 0.001
- link R_finger_right: geometry collision mesh filename=meshes/R_finger_right.stl scale=0.001 0.001 0.001; visual mesh filename=meshes/R_finger_right.stl scale=0.001 0.001 0.001
- link R_gripper_base: geometry collision mesh filename=meshes/R_gripper_base.stl scale=0.001 0.001 0.001; visual mesh filename=meshes/R_gripper_base.stl scale=0.001 0.001 0.001
- link R_link1: geometry collision mesh filename=meshes/R_link1.stl scale=0.001 0.001 0.001; visual mesh filename=meshes/R_link1.stl scale=0.001 0.001 0.001
- link R_link2: geometry collision mesh filename=meshes/R_link2.stl scale=0.001 0.001 0.001; visual mesh filename=meshes/R_link2.stl scale=0.001 0.001 0.001
- link R_link3: geometry collision mesh filename=meshes/R_link3.stl scale=0.001 0.001 0.001; visual mesh filename=meshes/R_link3.stl scale=0.001 0.001 0.001
- link R_link4: geometry collision mesh filename=meshes/R_link4.stl scale=0.001 0.001 0.001; visual mesh filename=meshes/R_link4.stl scale=0.001 0.001 0.001
- link R_link5: geometry collision mesh filename=meshes/R_link5.stl scale=0.001 0.001 0.001; visual mesh filename=meshes/R_link5.stl scale=0.001 0.001 0.001
- link R_link6: geometry collision mesh filename=meshes/R_link6.stl scale=0.001 0.001 0.001; visual mesh filename=meshes/R_link6.stl scale=0.001 0.001 0.001
- link R_link7: geometry collision mesh filename=meshes/R_link7.stl scale=0.001 0.001 0.001; visual mesh filename=meshes/R_link7.stl scale=0.001 0.001 0.001
- link R_shoulder_mount: mass 0.05 -> None; geometry 
Joints:
- joint L_gripper_base_fixed: origin xyz=0 0 0 rpy=0 0 0 -> xyz=0 0 -0.07 rpy=0 0 0
- joint L_gripper_joint: origin xyz=0 0.01836 -0.09 rpy=0 0 0 -> xyz=0 0.01836 -0.0205 rpy=0 0 0
- joint L_gripper_mimic: origin xyz=0 -0.01836 -0.09 rpy=0 0 0 -> xyz=0 -0.01836 -0.0205 rpy=0 0 0
- joint L_joint3: origin xyz=0 0 -0.0825 rpy=0 0 0 -> xyz=0.0155 0 -0.0825 rpy=0 0 0
- joint L_tcp_fixed: origin xyz=0 0 -0.175 rpy=0 0 0 -> xyz=0 0 -0.1055 rpy=0 0 0
- joint R_gripper_base_fixed: origin xyz=0 0 0 rpy=0 0 0 -> xyz=0 0 -0.07 rpy=0 0 0
- joint R_gripper_joint: origin xyz=0 0.01836 -0.09 rpy=0 0 0 -> xyz=0 0.01836 -0.0205 rpy=0 0 0
- joint R_gripper_mimic: origin xyz=0 -0.01836 -0.09 rpy=0 0 0 -> xyz=0 -0.01836 -0.0205 rpy=0 0 0
- joint R_joint3: origin xyz=0 0 -0.0825 rpy=0 0 0 -> xyz=0.0155 0 -0.0825 rpy=0 0 0
- joint R_tcp_fixed: origin xyz=0 0 -0.175 rpy=0 0 0 -> xyz=0 0 -0.1055 rpy=0 0 0
